Commit message: files updated for mockup

File: mockup_ws/src/fourze_vehicle_description/urdf/4ze_vehicle.urdf.xacro (robot description, xacro)
@@ -136,3 +136,37 @@
     <origin xyz="-0.82 0 0.15" rpy="0 ${pi/2} 0"/>
   </joint>
+  <!-- Accelerator pedal -->
+  <link name="accelerator_pedal">
+    <visual>
+      <origin xyz="0 0 0.11" rpy="0 0 0"/>
+      <geometry>
+        <box size="0.10 0.045 0.22"/>
+      </geometry>
+      <material name="motor_material"/>
+    </visual>
+  </link>
+  <joint name="accelerator_joint" type="revolute">
+    <parent link="base_link"/>
+    <child link="accelerator_pedal"/>
+    <origin xyz="0.48 -0.12 0.18" rpy="0 0 0"/>
+    <axis xyz="0 1 0"/>
+    <limit lower="0.0" upper="0.50" effort="10.0" velocity="2.0"/>
+  </joint>
+  <!-- Brake pedal -->
+  <link name="brake_pedal">
+    <visual>
+      <origin xyz="0 0 0.11" rpy="0 0 0"/>
+      <geometry>
+        <box size="0.10 0.055 0.22"/>
+      </geometry>
+      <material name="battery_material"/>
+    </visual>
+  </link>
+  <joint name="brake_joint" type="revolute">
+    <parent link="base_link"/>
+    <child link="brake_pedal"/>
+    <origin xyz="0.48 0.12 0.18" rpy="0 0 0"/>
+    <axis xyz="0 1 0"/>
+    <limit lower="0.0" upper="0.50" effort="10.0" velocity="2.0"/>
+  </joint>
 </robot>
